Commit message: updated launch files

File: urdf/exo_with_human.xacro (robot description, xacro)
@@ -8,10 +8,10 @@
   <xacro:include filename="depth_cameras_setup.xacro" />
   <xacro:include filename="human_dummy.xacro" />
-    <link name="world"/>
-    <joint name="pole_to_waist" type="fixed">
-        <parent link="world" />
-        <child link="waist_link" />
-        <origin xyz="0 0 0" rpy="0 0 0"/>
-    </joint>
+  <link name="world"/>
+  <joint name="pole_to_waist" type="fixed">
+      <parent link="world" />
+      <child link="waist_link" />
+      <origin xyz="0 0 0" rpy="0 0 0"/>
+  </joint>
   <link name="human_waist_link">
     <visual>
